File: Training_Hardware/Training_Hardware.kicad_pcb (KiCad board)
At the start: 2 copper layers, 102.1 x 43.2 mm, 17 parts, among them J1 RJ45_LED_Shielded, U1 Teensy4.1_DEV-16771, U2 OKI, U3 ATA6561-GBQW-N

Commit message: PCB edits
Other:
- outline, holes or cut-outs redrawn
Changed lines of the file:
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@@
 	)
 	(gr_rect
-		(start 38.1 40.64)
-		(end 140.208 83.82)
+		(start 38.1 42.687692)
+		(end 140.18054 83.82)
 		(stroke
 			(width 0.05)
@@
 		(min_thickness 0.1778)
 		(filled_areas_thickness no)
-		(fill yes
+		(fill
 			(thermal_gap 0.5)
 			(thermal_bridge_width 0.5)
