File: training_hardware/CAN.kicad_sch (KiCad schematic)
At the start: 5 parts, among them U2 ATA6561-GBQW-N

Commit message: pp
Parts:
- removed U2: ATA6561-GBQW-N, VDFN8_3X3_MCH, symbol 2026_training_hardware:ATA6561-GBQW-N
- added U2: ATA6561-GAQW, 2026Training_Hardware:SOIC8_4P9X3P9MC_MCH-L, symbol 2026_training_hardware:ATA6561-GAQW
- C4, C5: footprint (none) -> Capacitor_SMD:C_0603_1608Metric_Pad1.08x0.95mm_HandSolder
- Conn1: footprint (none) -> MRDT_Connectors:MOLEX_SL_02_Vertical
- R3: footprint (none) -> Resistor_SMD:R_0603_1608Metric_Pad0.98x0.95mm_HandSolder
Connections:
- net +3V3: now also U2.5 (VIO)
- net +5V: now also U2.3 (VCC)
- net GND: now also U2.2 (GND)
- net RXD: now also U2.4 (RXD)
- net STBY: now also U2.8 (STBY)
- net TXD: now also U2.1 (TXD)
- net at Conn1.2, R3.2: now also U2.6 (CANL)
- net at Conn1.1, R3.1: now also U2.7 (CANH)
Other:
- moved on the sheet: C5, Conn1, R3
