File: training_hardware/MCU.kicad_sch (KiCad schematic)
At the start: 3 parts, among them J1 RJ45_LED_Shielded, U1 Teensy4.1_DEV-16771

Commit message: Finished layout training
Parts:
- C3: footprint (none) -> Capacitor_SMD:C_0603_1608Metric_Pad1.08x0.95mm_HandSolder
- J1: footprint (none) -> MRDT_Connectors:RJ45_Teensy
- U1: footprint MODULE_DEV-16771 -> MRDT_Shields:Teensy_4_1_Ethernet
Connections:
- net +5V: now also U1.VIN
- no-connect marks 3 -> 14
Changed lines of the file:
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@@
+	)
+	(no_connect
+		(at 163.83 83.82)
+	)
+	(no_connect
+		(at 163.83 93.98)
 	)
 	(no_connect
@@
 	)
 	(no_connect
+		(at 163.83 58.42)
+	)
+	(no_connect
+		(at 163.83 105.41)
+	)
+	(no_connect
+		(at 163.83 106.68)
+	)
+	(no_connect
+		(at 163.83 104.14)
+	)
+	(no_connect
 		(at 214.63 40.64)
 	)
+	(no_connect
+		(at 163.83 91.44)
+	)
+	(no_connect
+		(at 163.83 96.52)
+	)
+	(no_connect
+		(at 163.83 81.28)
+	)
+	(no_connect
+		(at 163.83 60.96)
+	)
+	(no_connect
+		(at 163.83 101.6)
+	)
 	(wire
 		(pts
@@
 	(wire
 		(pts
+			(xy 114.3 55.88) (xy 114.3 66.04)
+		)
+		(stroke
+			(width 0)
+			(type default)
+		)
+	)
+	(wire
+		(pts
 			(xy 222.25 60.96) (xy 222.25 63.5)
 		)
@@
 		(pts
 			(xy 241.3 38.1) (xy 241.3 39.37)
+		)
+		(stroke
+			(width 0)
+			(type default)
+		)
+	)
+	(wire
+		(pts
+			(xy 114.3 66.04) (xy 123.19 66.04)
 		)
 		(stroke
@@
 			)
 		)
-		(property "Footprint" ""
+		(property "Footprint" "MRDT_Connectors:RJ45_Teensy"
 			(at 220.345 50.8 90)
 			(effects
@@
 	)
 	(symbol
+		(lib_id "power:+5V")
+		(at 114.3 55.88 0)
+		(unit 1)
+		(exclude_from_sim no)
+		(in_bom yes)
+		(on_board yes)
+		(dnp no)
+		(fields_autoplaced yes)
+		(property "Reference" "#PWR017"
+			(at 114.3 59.69 0)
+			(effects
+				(font
+					(size 1.27 1.27)
+				)
+				(hide yes)
+			)
+		)
+		(property "Value" "+5V"
+			(at 114.3 50.8 0)
+			(effects
+				(font
+					(size 1.27 1.27)
+				)
+			)
+		)
+		(property "Footprint" ""
+			(at 114.3 55.88 0)
+			(effects
+				(font
+					(size 1.27 1.27)
+				)
+				(hide yes)
+			)
+		)
+		(property "Datasheet" ""
+			(at 114.3 55.88 0)
+			(effects
+				(font
+					(size 1.27 1.27)
+				)
+				(hide yes)
+			)
+		)
+		(property "Description" "Power symbol creates a global label with name \"+5V\""
+			(at 114.3 55.88 0)
+			(effects
+				(font
+					(size 1.27 1.27)
+				)
+				(hide yes)
+			)
+		)
+		(pin "1"
+		)
+		(instances
+			(project "training_hardware"
+				(path "/19aa0e78-5ab4-46df-84c9-9ca161187559/7e06b3c1-2423-42b6-bbd6-08ed46d7df02"
+					(reference "#PWR017")
+					(unit 1)
+				)
+			)
+		)
+	)
+	(symbol
 		(lib_id "power:GND")
 		(at 171.45 153.67 0)
@@
 			)
 		)
-		(property "Footprint" ""
+		(property "Footprint" "Capacitor_SMD:C_0603_1608Metric_Pad1.08x0.95mm_HandSolder"
 			(at 215.5952 78.74 0)
 			(effects
@@
 			)
 		)
-		(property "Footprint" "MODULE_DEV-16771"
+		(property "Footprint" "MRDT_Shields:Teensy_4_1_Ethernet"
 			(at 196.85 109.22 0)
 			(effects
