File: training_hardware/MCU.kicad_sch (KiCad schematic)
At the start: 3 parts, among them J1 RJ45_LED_Shielded, U1 Teensy4.1_DEV-16771

Commit message: pp
Parts:
- C3: footprint (none) -> Capacitor_SMD:C_0603_1608Metric_Pad1.08x0.95mm_HandSolder
- J1: footprint (none) -> MRDT_Connectors:RJ45_Teensy
- U1: footprint MODULE_DEV-16771 -> MRDT_Shields:Teensy_4_1_Ethernet
Changed lines of the file:
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@@
 			)
 		)
-		(property "Footprint" ""
+		(property "Footprint" "MRDT_Connectors:RJ45_Teensy"
 			(at 220.345 50.8 90)
 			(effects
@@
 			)
 		)
-		(property "Footprint" ""
+		(property "Footprint" "Capacitor_SMD:C_0603_1608Metric_Pad1.08x0.95mm_HandSolder"
 			(at 215.5952 78.74 0)
 			(effects
@@
 			)
 		)
-		(property "Footprint" "MODULE_DEV-16771"
+		(property "Footprint" "MRDT_Shields:Teensy_4_1_Ethernet"
 			(at 196.85 109.22 0)
 			(effects
