File: training_hardware/training_hardware.kicad_sch (KiCad schematic)
At the start: 0 parts

Commit message: pp
Parts:
- added H1, H2, H3, H4: MountingHole, MRDT_Drill_Holes:4_40_Hole, symbol Mechanical:MountingHole
